File: hardware/MAX31855K_Breakout/MAX31855K_Breakout.kicad_sch (KiCad schematic)
At the start: 19 parts, among them J1 Temperature Probe Connector, J2 SSR Connector, J3 SPI Connector, Q1 Q_NMOS_GSD, U1 MAX31855KASA, U2 TPS631000

Commit message: chore: lint hardware (#12)
Parts:
- U2: symbol User:TPS631000 -> Reflow_Oven:TPS631000; DigiKey Part Number 296-TPS631000DRLRCT-ND -> (none)
Connections:
- net GND: now also USB_C1.S1 (Shield)
Changed lines of the file:
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@@
 	(title_block
 		(title "MAX31855K Breakout")
-		(date "2025-11-29")
-		(rev "v3.0.1")
+		(date "2025-12-01")
+		(rev "v3.0.2")
 		(company "Cory Buecker")
 		(comment 1 "© 2025 Stanton Cory Buecker")
@@
 		(pts
 			(xy 69.85 64.77) (xy 69.85 63.5)
+		)
+		(stroke
+			(width 0)
+			(type default)
+		)
+	)
+	(wire
+		(pts
+			(xy 73.66 64.77) (xy 73.66 63.5)
 		)
 		(stroke
@@
 		)
 		(property "DigiKey Part Number" "MAX31855KASA+TCT-ND"
-			(at 198.12 107.95 0)
+			(at 213.36 123.19 0)
 			(effects
 				(font
@@
 				(path "/a793c5ac-b66c-4259-9d59-43bd772bada2"
 					(reference "U1")
+					(unit 1)
+				)
+			)
+		)
+	)
+	(symbol
+		(lib_id "power:GND")
+		(at 73.66 64.77 0)
+		(unit 1)
+		(exclude_from_sim no)
+		(in_bom yes)
+		(on_board yes)
+		(dnp no)
+		(fields_autoplaced yes)
+		(property "Reference" "#PWR014"
+			(at 73.66 71.12 0)
+			(effects
+				(font
+					(size 1.27 1.27)
+				)
+				(hide yes)
+			)
+		)
+		(property "Value" "GND"
+			(at 73.66 69.85 0)
+			(effects
+				(font
+					(size 1.27 1.27)
+				)
+			)
+		)
+		(property "Footprint" ""
+			(at 73.66 64.77 0)
+			(effects
+				(font
+					(size 1.27 1.27)
+				)
+				(hide yes)
+			)
+		)
+		(property "Datasheet" ""
+			(at 73.66 64.77 0)
+			(effects
+				(font
+					(size 1.27 1.27)
+				)
+				(hide yes)
+			)
+		)
+		(property "Description" "Power symbol creates a global label with name \"GND\" , ground"
+			(at 73.66 64.77 0)
+			(effects
+				(font
+					(size 1.27 1.27)
+				)
+				(hide yes)
+			)
+		)
+		(pin "1"
+		)
+		(instances
+			(project "MAX31855K_Breakout"
+				(path "/a793c5ac-b66c-4259-9d59-43bd772bada2"
+					(reference "#PWR014")
 					(unit 1)
 				)
@@
 		(pin "A9"
 		)
+		(pin "S1"
+		)
 		(instances
 			(project ""
@@
 	)
 	(symbol
-		(lib_id "User:TPS631000")
+		(lib_id "Reflow_Oven:TPS631000")
 		(at 100.33 104.14 0)
 		(unit 1)
@@
 		(dnp no)
 		(property "Reference" "U2"
-			(at 108.204 90.17 0)
+			(at 100.33 104.14 0)
 			(effects
 				(font
@@
 		)
 		(property "Value" "TPS631000"
-			(at 112.522 92.71 0)
+			(at 86.36 115.57 0)
 			(effects
 				(font
@@
 			(effects
 				(font
-					(size 1.27 1.27)
-				)
-				(hide yes)
-			)
-		)
-		(property "DigiKey Part Number" "296-TPS631000DRLRCT-ND"
-			(at 100.33 104.14 0)
-			(effects
-				(font
