File: hardware/MCP9601-Sensor/MCP9601-Sensor.kicad_pcb (KiCad board)
At the start: 2 copper layers, 47 x 35 mm, 30 parts, among them J1 Conn_01x02_Pin, J2 Conn_01x02_Pin, J3 Conn_01x02_Pin, J4 Conn_01x04_Pin, Q1 BSS138, U1 MCP9601

Commit message: feat: implement software with ESP32 C6
Add USB-C breakout design for power and data
Other:
- board text added: "${TITLE} ${REVISION} ${COMPANY}"
